File: Hardware/KiCad/acer-core/acer-core.kicad_sch (KiCad schematic)
At the start: 26 parts, among them J1 USB_C_Receptacle_USB2.0_16P, J2 Conn_01x10_Pin, J3 Conn_01x10_Pin, J4 Conn_01x16_Socket, Q1 AO3401A, SW1 RESET, SW2 USER, U1 ESP32-S3-WROOM-1, U2 USBLC6-2SC6, U3 WIO-SX1262, U4 TLV75733PDBV

Commit message: Routing Done
Parts:
- removed C5, C6: 10uF, Capacitor_SMD:C_0805_2012Metric, symbol Device:C
- removed D2: 1N5817W, Diode_SMD:D_SOD-123, symbol Diode:1N5817
- removed J1: USB_C_Receptacle_USB2.0_16P, SB-Lib:CUI_UJ20-C-V-C-3-SMT-TR, symbol Connector:USB_C_Receptacle_USB2.0_16P
- removed J2, J3: Conn_01x10_Pin, Connector_PinHeader_2.54mm:PinHeader_1x10_P2.54mm_Vertical, symbol Connector:Conn_01x10_Pin
- removed J4: Conn_01x16_Socket, Connector_PinHeader_2.54mm:PinHeader_1x16_P2.54mm_Vertical, symbol Connector:Conn_01x16_Socket
- removed Q1: AO3401A, Package_TO_SOT_SMD:SOT-23, symbol Transistor_FET:AO3401A
- removed R2: 5K1, Resistor_SMD:R_0603_1608Metric, symbol Device:R_US
- removed R5: 100K, Resistor_SMD:R_0603_1608Metric, symbol Device:R_US
- removed U2: USBLC6-2SC6, Package_TO_SOT_SMD:SOT-23-6, symbol Power_Protection:USBLC6-2SC6
- removed U3: WIO-SX1262, SB-Lib:Wio-SX1262-SB, symbol SB-Lib:MODULE-WIO-SX1262-SB
- removed U4: TLV75733PDBV, Package_TO_SOT_SMD:SOT-23-5, symbol Regulator_Linear:TLV75733PDBV
- added J1, J2: Conn_01x14_Pin, Connector_PinHeader_2.54mm:PinHeader_1x14_P2.54mm_Vertical, symbol Connector:Conn_01x14_Pin
- added U2: WIO-SX1262, SB_RF_Module:Wio-SX1262-SB, symbol SB_RF_Module:WIO-SX1262-SB
- C1: MPN (none) -> GRM21BR71A106KA73L; Manufacturer (none) -> Murata; Supplier (none) -> Digikey; Supplier_PN (none) -> 490-10516-1-ND
- C2: MPN (none) -> CL10B104JB8NNNC; Manufacturer (none) -> Samsung; Supplier (none) -> Digikey; Supplier_PN (none) -> 1276-1033-1-ND
- C3: renamed from C7; MPN (none) -> CL10B104JB8NNNC; Manufacturer (none) -> Samsung; Supplier (none) -> Digikey; Supplier_PN (none) -> 1276-1033-1-ND
- C4: renamed from C8; MPN (none) -> CL10B104JB8NNNC; Manufacturer (none) -> Samsung; Supplier (none) -> Digikey; Supplier_PN (none) -> 1276-1033-1-ND
- C5: renamed from C3; MPN (none) -> GRM21BR71A106KA73L; Manufacturer (none) -> Murata; Supplier (none) -> Digikey; Supplier_PN (none) -> 490-10516-1-ND
- C6: renamed from C4; MPN (none) -> CL10B104JB8NNNC; Manufacturer (none) -> Samsung; Supplier (none) -> Digikey; Supplier_PN (none) -> 1276-1033-1-ND
- D1: value Blue 2.9V -> Green 2.1V; MPN (none) -> LTST-C190GKT; Manufacturer (none) -> Lite-On; Supplier (none) -> Digikey; Supplier_PN (none) -> 160-LTST-C190GKTCT-ND
- R1: MPN (none) -> CRCW060310K0FKEA; Manufacturer (none) -> Vishay Dale; Supplier (none) -> Digikey; Supplier_PN (none) -> 541-10.0KHCT-ND
- R2: renamed from R4; value 330 -> 130; MPN (none) -> RC0603FR-07130RL; Manufacturer (none) -> YAGEO; Supplier (none) -> Digikey; Supplier_PN (none) -> 311-130HRCT-ND
- R3: value 5K1 -> 10K; MPN (none) -> CRCW060310K0FKEA; Manufacturer (none) -> Vishay Dale; Supplier (none) -> Digikey; Supplier_PN (none) -> 541-10.0KHCT-ND
- SW1, SW2: footprint SB-Lib:B3U-1000P -> SB_Button_Switch_SMD:SW_SKRPABE010; MPN (none) -> SKRPABE010; Manufacturer (none) -> Alps Alpine; Supplier (none) -> Digikey; Supplier_PN (none) -> 4809-SKRPABE010CT-ND
Connections:
- net +3.3V: now also R3.2, J1.1 (Pin_1), U2.8 (VCC)
- net EN: now also J1.2 (Pin_2)
- net GND: now also J1.9 (Pin_9), J2.5 (Pin_5), U2.10 (GND2), U2.7 (GND1); no longer R3.2
- net IO1: now also J2.1 (Pin_1)
- net IO12: now also J2.13 (Pin_13)
- net IO13: now also J2.12 (Pin_12)
- net IO14: now also J2.11 (Pin_11)
- net IO15: now also J1.10 (Pin_10)
- net IO16: now also J1.11 (Pin_11)
- net IO17: now also J1.12 (Pin_12)
- net IO18: now also J1.13 (Pin_13)
- net IO2: now also J2.2 (Pin_2)
- net IO3: now also J1.14 (Pin_14)
- net IO4: now also J1.3 (Pin_3)
- net IO5: now also J1.4 (Pin_4)
- net LORA_BUSY: now also U2.11 (BUSY)
- net LORA_DIO: now also U2.12 (DIO1)
- net LORA_MISO: now also U2.2 (MISO)
- net LORA_MOSI: now also U2.3 (MOSI)
- net LORA_NSS: now also U2.6 (NSS)
- net LORA_RF_SW1: now also U2.1 (RF_SW1)
- net LORA_RST: now also R3.1, U2.5 (RST)
- net LORA_SCK: now also U2.4 (SCK)
- net RXD0: now also J2.4 (Pin_4)
- net TXD0: now also J2.3 (Pin_3)
- net USB_D+: now also J1.8 (Pin_8)
- net USB_D-: now also J1.7 (Pin_7)
- net USER: now also J2.6 (Pin_6)
- net IO46: now reaches U1.16 (IO46)
- net IO46: now also J2.8 (Pin_8)
- net IO11: now reaches U1.19 (IO11)
- net IO11: now also J2.14 (Pin_14)
- net IO21: now reaches U1.23 (IO21)
- net IO21: now also J2.10 (Pin_10)
- net IO47: now reaches U1.24 (IO47)
- net IO47: now also J2.9 (Pin_9)
- net IO45: now reaches U1.26 (IO45)
- net IO45: now also J2.7 (Pin_7)
- net IO6: now reaches U1.6 (IO6)
- net IO6: now also J1.5 (Pin_5)
- net IO7: now reaches U1.7 (IO7)
- net IO7: now also J1.6 (Pin_6)
- no-connect marks 13 -> 4
Other:
- note removed: "Power Supply"
- note removed: "USB / UART / JTAG"
- moved on the sheet: C5, C6

Commit message: Some fixes
Parts:
- U1: value ESP32-S3-WROOM-1 -> ESP32-S3-WROOM-1-N4; MPN (none) -> ESP32-S3-WROOM-1-N4; Manufacturer (none) -> Espressif; Supplier (none) -> Digikey; Supplier_PN (none) -> 1965-ESP32-S3-WROOM-1-N4CT-ND
- U2: MPN (none) -> 114993390; Manufacturer (none) -> Seeed; Supplier (none) -> Digikey; Supplier_PN (none) -> 1597-114993390CT-ND
Connections:
- net IO15: now also J1.7 (Pin_7); no longer J1.10 (Pin_10)
- net IO16: now also J1.8 (Pin_8); no longer J1.11 (Pin_11)
- net IO17: now also J1.10 (Pin_10); no longer J1.12 (Pin_12)
- net IO18: now also J1.11 (Pin_11); no longer J1.13 (Pin_13)
- net IO3: now also J2.14 (Pin_14); no longer J1.14 (Pin_14)
- net IO45: now also J2.12 (Pin_12); no longer J2.7 (Pin_7)
- net IO46: now also J2.13 (Pin_13); no longer J2.8 (Pin_8)
- net LORA_BUSY: now also U1.19 (IO11); no longer U1.33 (IO40)
- net LORA_DIO: now also U1.24 (IO47); no longer U1.32 (IO39)
- net LORA_MISO: now also U1.22 (IO14); no longer U1.17 (IO9)
- net LORA_MOSI: now also U1.21 (IO13); no longer U1.18 (IO10)
- net LORA_NSS: now also U1.17 (IO9); no longer U1.34 (IO41)
- net LORA_RF_SW1: now also U1.23 (IO21); no longer U1.31 (IO38)
- net LORA_SCK: now also U1.20 (IO12); no longer U1.12 (IO8)
- net USB_D+: now also J1.14 (Pin_14); no longer J1.8 (Pin_8)
- net USB_D-: now also J1.13 (Pin_13); no longer J1.7 (Pin_7)
- net USER: now also J2.11 (Pin_11); no longer J2.6 (Pin_6)
- removed net IO11: J2.14 (Pin_14), U1.19 (IO11)
- removed net IO12: J2.13 (Pin_13), U1.20 (IO12)
- removed net IO13: J2.12 (Pin_12), U1.21 (IO13)
- removed net IO14: J2.11 (Pin_11), U1.22 (IO14)
- net IO21 renamed IO38
- net IO38: now also U1.31 (IO38); no longer U1.23 (IO21)
- net IO47 renamed IO39
- net IO39: now also U1.32 (IO39); no longer U1.24 (IO47)
- net LORA_RST renamed ~{LORA_RST}
- net ~{LORA_RST}: now also U1.18 (IO10); no longer U1.35 (IO42)
- new net IO40: J2.8 (Pin_8), U1.33 (IO40)
- new net IO41: J2.7 (Pin_7), U1.34 (IO41)
- new net IO42: J2.6 (Pin_6), U1.35 (IO42)
- new net IO8: J1.12 (Pin_12), U1.12 (IO8)

Commit message: Routing Done
Parts:
- removed SW1: RESET, SB_Button_Switch_SMD:SW_SKRPABE010, symbol Switch:SW_Push
- removed SW2: USER, SB_Button_Switch_SMD:SW_SKRPABE010, symbol Switch:SW_Push
- added C7: 1uF, Capacitor_SMD:C_0603_1608Metric, symbol Device:C
- added S1: RESET, SB_Button_Switch_SMD:SW_SKRPABE010, symbol SB_Button_Switch_SMD:SKRPABE010
- added S2: USER, SB_Button_Switch_SMD:SW_SKRPABE010, symbol SB_Button_Switch_SMD:SKRPABE010
Connections:
- net EN: now also C7.1, S1.1, S1.2
- net GND: now also J1.10 (Pin_10), J2.10 (Pin_10), C7.2, S1.3, S1.4, S2.3, S2.4; no longer J1.9 (Pin_9), J2.5 (Pin_5)
- net IO15: now also J1.9 (Pin_9); no longer J1.7 (Pin_7)
- net IO16: now also J1.11 (Pin_11); no longer J1.8 (Pin_8)
- net IO17: now also J1.12 (Pin_12); no longer J1.10 (Pin_10)
- net IO18: now also J1.13 (Pin_13); no longer J1.11 (Pin_11)
- net IO38: now also J2.9 (Pin_9); no longer J2.10 (Pin_10)
- net IO39: now also J2.8 (Pin_8); no longer J2.9 (Pin_9)
- net IO40: now also J2.7 (Pin_7); no longer J2.8 (Pin_8)
- net IO41: now also J2.6 (Pin_6); no longer J2.7 (Pin_7)
- net IO42: now also J2.5 (Pin_5); no longer J2.6 (Pin_6)
- net IO8: now also J1.14 (Pin_14); no longer J1.12 (Pin_12)
- net USB_D+: now also J1.8 (Pin_8); no longer J1.14 (Pin_14)
- net USB_D-: now also J1.7 (Pin_7); no longer J1.13 (Pin_13)
- net USER: now also S2.1, S2.2
Other:
- moved on the sheet: R1
